File: Modulo_ENC28J60.kicad_pcb (KiCad board)
At the start: 2 copper layers, 66.4 x 33.6 mm, 21 parts, among them J1 Conn_02x06_Odd_Even, J2 RJ45_Bel_SI-60062-F, U1 ENC28J60x-SO, Y1 25Mhz

Commit message: Roteamento de trilhas
Routing:
- net GNDREF: track 0.00 -> 216.7 mm, vias 0 -> 1
- net +3.3V: track 0.00 -> 99.6 mm, vias 0 -> 3
- net LEDB: track 0.00 -> 69.4 mm, vias 0 -> 1
- net TD+: track 0.00 -> 46.1 mm, vias 0 -> 1
- net RD-: track 0.00 -> 45.2 mm
- net LEDA: track 0.00 -> 44.2 mm
- net RD+: track 0.00 -> 37.5 mm
- net TD-: track 0.00 -> 36.5 mm
- net TCT: track 0.00 -> 29.5 mm, vias 0 -> 1
- net MISO: track 0.00 -> 21.9 mm, vias 0 -> 1
- net Net-(C2-Pad2): track 0.00 -> 20.3 mm
- net Net-(C1-Pad2): track 0.00 -> 16.9 mm
- net MOSI: track 0.00 -> 15.9 mm, vias 0 -> 1
- net unconnected-(J2-PadSH): track 0.00 -> 15.5 mm
- net SCK: track 0.00 -> 15.3 mm
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